File: cwbpf.kicad_sch (KiCad schematic)
At the start: 35 parts, among them J1 AudioJack4, J2 AudioJack4, U1 NJM4580, U2 NJM4580, U3 MCP4921

Commit message: v0.0.1
Parts:
- removed RV3: 10k, symbol Device:R_Potentiometer
- added RV3: 10k, Library:基板取付用ボリューム つまみ付き 薄型 10kΩ 2連, symbol Library:基板取付用ボリューム つまみ付き 薄型 2連
- A1: footprint Module:RaspberryPi_Pico_Common_Unspecified -> Library:RaspberryPi_Pico_slim
- C1, C2, C3, C8: footprint (none) -> Capacitor_THT:C_Disc_D7.5mm_W2.5mm_P5.00mm
- C10: footprint (none) -> Capacitor_THT:CP_Radial_D8.0mm_P3.50mm
- C4, C5, C6, C7: footprint (none) -> Capacitor_THT:C_Disc_D7.0mm_W2.5mm_P5.00mm
- C9: footprint (none) -> Capacitor_THT:CP_Radial_D5.0mm_P2.00mm
- J1, J2: footprint (none) -> Connector_Audio:Jack_3.5mm_PJ320E_Horizontal
- R1, R10, R11, R12, R13, R14, R15, R2, R3, R4, R5, R6, R7, R8, R9: footprint (none) -> Resistor_THT:R_Axial_DIN0204_L3.6mm_D1.6mm_P5.08mm_Horizontal
- RV1, RV2, RV4: footprint (none) -> Library:基板取付用ボリューム つまみ付き 薄型 10kΩ 2連; symbol Device:R_Potentiometer -> Library:基板取付用ボリューム つまみ付き 薄型 2連
- U1, U2: footprint (none) -> Package_SIP:SIP-8_19x3mm_P2.54mm
- U3: footprint (none) -> Package_DIP:DIP-8_W7.62mm
Connections:
- net +3.3V: now also RV2.5 (R1_3), RV3.1 (R12_1); no longer RV2.1
- net AGND: now also RV1.1 (R12_1), RV2.1 (R12_1), RV4.5 (R1_3), RV3.5 (R1_3); no longer RV1.3
- net GND: no longer RV2.3, RV4.3
- net GPIO_28: now also RV3.2 (R1_2)
- net at R1.1: now also RV1.5 (R1_3); no longer RV1.1
- no-connect marks 3 -> 36
Other:
- note added: "基板取付用ボリューム つまみ付き 薄型 10kΩA 2連"
- note added: "基板取付用ボリューム つまみ付き 薄型 10kΩB 2連"
- moved on the sheet: C1, C10, C3, C4, C5, C6, C7, C8, J1, J2, R1, R14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
